Commit message: refactor(B-001): move URDF into non-exec package + resolve KDL physics issue w/ base link

File: ros2_ws/src/robot_description/urdf/chassis_model.xacro (robot description, xacro)
@@ -1,5 +1,5 @@
 <?xml version="1.0" ?>
 <robot name="chassis_model" xmlns:xacro="http://www.ros.org/wiki/xacro">
-<xacro:include filename="$(find chassis_description)/urdf/materials.xacro" />
+<xacro:include filename="$(find robot_description)/urdf/materials.xacro" />
 <xacro:arg name="controllers_yaml" default="" />
 <xacro:arg name="controllers_sim_yaml" default="" />
@@ -8,4 +8,11 @@
 <!--xacro:include filename="$(find chassis_description)/urdf/chassis_model.trans" /-->
 <!--xacro:include filename="$(find chassis_description)/urdf/chassis_model.gazebo" /-->
+<!-- New dummy root link with no inertia so KDL as a root node w/ no inertia while base_link still keeps physics intact-->
+<link name="base_dummy"/>
+<joint name="base_link" type="fixed">
+  <parent link="base_dummy"/>
+  <child link="base_link"/>
+  <origin xyz="0 0 0" rpy="0.0 0.0 0.0"/>
+</joint>
 <link name="base_link">
   <inertial>
