Commit message: feat(B-002): fix transform issues with urdf file + add bridging with ign gz topics and ros2 topics

File: ros2_ws/src/robot_description/urdf/robot_core.urdf.xacro (robot description, xacro)
@@ -11,14 +11,15 @@
     <parent link="base_footprint"/>
     <child link="base_link"/>
-    <origin rpy="0.0 0.0 0.0" xyz="0 0 0.359"/>
+    <!-- base_link is located midway between the two centre wheel axes. -->
+    <origin rpy="0.0 0.0 0.0" xyz="0.3624 0 0.115"/>
   </joint>
   <link name="base_link">
     <inertial>
-      <origin rpy="0 0 0" xyz="0.3026093095883329 4.957188589394069e-17 -0.00019403432456449078"/>
+      <origin rpy="0 0 0" xyz="-0.0597906904116671 4.957188589394069e-17 0.2438059656754355"/>
       <mass value="368.7010327977625"/>
       <inertia ixx="7.357137" ixy="-0.0" ixz="-0.006189" iyy="12.009665" iyz="-0.0" izz="17.59793"/>
     </inertial>
     <visual>
-      <origin rpy="0 0 0" xyz="0 0 0"/>
+      <origin rpy="0 0 ${pi}" xyz="0.3624 0 0.244"/>
       <geometry>
         <mesh filename="package://robot_description/meshes/base_link.stl" scale="0.001 0.001 0.001"/>
@@ -27,5 +28,5 @@
     </visual>
     <collision>
-      <origin rpy="0 0 0" xyz="0 0 0"/>
+      <origin rpy="0 0 ${pi}" xyz="0.3624 0 0.244"/>
       <geometry>
         <mesh filename="package://robot_description/meshes/base_link.stl" scale="0.001 0.001 0.001"/>
@@ -33,5 +34,5 @@
     </collision>
   </link>
-  <link name="suspension_1_left_1">
+  <link name="suspension_1_right_1">
     <inertial>
       <origin rpy="0 0 0" xyz="-0.06679854886170258 -0.019220268351824554 -0.09147358690967579"/>
@@ -53,5 +54,5 @@
     </collision>
   </link>
-  <link name="suspension_1_right_1">
+  <link name="suspension_1_left_1">
     <inertial>
       <origin rpy="0 0 0" xyz="-0.06679854886170233 0.019220268351824554 -0.09147358690967583"/>
@@ -73,5 +74,5 @@
     </collision>
   </link>
-  <link name="suspension_2_left_1">
+  <link name="suspension_2_right_1">
     <inertial>
       <origin rpy="0 0 0" xyz="-0.039308541684192844 0.019050000000000067 -0.062225074163904326"/>
@@ -93,5 +94,5 @@
     </collision>
   </link>
-  <link name="suspension_2_right_1">
+  <link name="suspension_2_left_1">
     <inertial>
       <origin rpy="0 0 0" xyz="-0.03930854168419273 -0.019050000000000122 -0.06222507416390427"/>
@@ -113,111 +114,111 @@
     </collision>
   </link>
+  <link name="wheel_r_3">
+    <inertial>
+      <origin rpy="0 0 0" xyz="-1.4432899320127035e-15 -0.05499999999999988 3.608224830031759e-16"/>
+      <mass value="35.77866096632706"/>
+      <inertia ixx="0.154692" ixy="-0.0" ixz="0.0" iyy="0.23723" iyz="-0.0" izz="0.154692"/>
+    </inertial>
+    <visual>
+      <origin rpy="0 0 0" xyz="-0.7524 0.281125 0.244"/>
+      <geometry>
+        <mesh filename="package://robot_description/meshes/wheel_3.stl" scale="0.001 0.001 0.001"/>
+      </geometry>
+      <material name="silver"/>
+    </visual>
+    <collision>
+      <origin rpy="0 0 0" xyz="-0.7524 0.281125 0.244"/>
+      <geometry>
+        <mesh filename="package://robot_description/meshes/wheel_3.stl" scale="0.001 0.001 0.001"/>
+      </geometry>
+    </collision>
+  </link>
+  <link name="wheel_r_2">
+    <inertial>
+      <origin rpy="0 0 0" xyz="-1.609823385706477e-15 -0.05499999999999988 1.3877787807814457e-16"/>
+      <mass value="35.77866096632706"/>
+      <inertia ixx="0.154692" ixy="0.0" ixz="0.0" iyy="0.23723" iyz="-0.0" izz="0.154692"/>
+    </inertial>
+    <visual>
+      <origin rpy="0 0 0" xyz="-0.3624 0.281125 0.244"/>
+      <geometry>
+        <mesh filename="package://robot_description/meshes/wheel_2.stl" scale="0.001 0.001 0.001"/>
+      </geometry>
+      <material name="silver"/>
+    </visual>
+    <collision>
+      <origin rpy="0 0 0" xyz="-0.3624 0.281125 0.244"/>
+      <geometry>
+        <mesh filename="package://robot_description/meshes/wheel_2.stl" scale="0.001 0.001 0.001"/>
+      </geometry>
+    </collision>
+  </link>
+  <link name="wheel_r_1">
+    <inertial>
+      <origin rpy="0 0 0" xyz="-1.7208456881689926e-15 -0.05499999999999988 1.1102230246251565e-16"/>
+      <mass value="35.77866096632706"/>
+      <inertia ixx="0.154692" ixy="-0.0" ixz="0.0" iyy="0.23723" iyz="-0.0" izz="0.154692"/>
+    </inertial>
+    <visual>
+      <origin rpy="0 0 0" xyz="0.1376 0.281125 0.244"/>
+      <geometry>
+        <mesh filename="package://robot_description/meshes/wheel_1.stl" scale="0.001 0.001 0.001"/>
+      </geometry>
+      <material name="silver"/>
+    </visual>
+    <collision>
+      <origin rpy="0 0 0" xyz="0.1376 0.281125 0.244"/>
+      <geometry>
+        <mesh filename="package://robot_description/meshes/wheel_1.stl" scale="0.001 0.001 0.001"/>
+      </geometry>
+    </collision>
+  </link>
+  <link name="wheel_1">
+    <inertial>
+      <origin rpy="0 0 0" xyz="-1.7208456881689926e-15 0.05499999999999988 1.942890293094024e-16"/>
+      <mass value="35.77866096632706"/>
+      <inertia ixx="0.154692" ixy="0.0" ixz="0.0" iyy="0.23723" iyz="0.0" izz="0.154692"/>
+    </inertial>
+    <visual>
+      <origin rpy="0 0 0" xyz="0.1376 -0.281125 0.244"/>
+      <geometry>
+        <mesh filename="package://robot_description/meshes/wheel_r_1.stl" scale="0.001 0.001 0.001"/>
+      </geometry>
+      <material name="silver"/>
+    </visual>
+    <collision>
+      <origin rpy="0 0 0" xyz="0.1376 -0.281125 0.244"/>
+      <geometry>
+        <mesh filename="package://robot_description/meshes/wheel_r_1.stl" scale="0.001 0.001 0.001"/>
+      </geometry>
+    </collision>
+  </link>
+  <link name="wheel_2">
+    <inertial>
+      <origin rpy="0 0 0" xyz="-1.609823385706477e-15 0.05499999999999988 2.220446049250313e-16"/>
+      <mass value="35.77866096632706"/>
+      <inertia ixx="0.154692" ixy="-0.0" ixz="0.0" iyy="0.23723" iyz="0.0" izz="0.154692"/>
+    </inertial>
+    <visual>
+      <origin rpy="0 0 0" xyz="-0.3624 -0.281125 0.244"/>
+      <geometry>
+        <mesh filename="package://robot_description/meshes/wheel_r_2.stl" scale="0.001 0.001 0.001"/>
+      </geometry>
+      <material name="silver"/>
+    </visual>
+    <collision>
+      <origin rpy="0 0 0" xyz="-0.3624 -0.281125 0.244"/>
+      <geometry>
+        <mesh filename="package://robot_description/meshes/wheel_r_2.stl" scale="0.001 0.001 0.001"/>
+      </geometry>
+    </collision>
+  </link>
   <link name="wheel_3">
     <inertial>
-      <origin rpy="0 0 0" xyz="-1.4432899320127035e-15 -0.05499999999999988 3.608224830031759e-16"/>
-      <mass value="35.77866096632706"/>
-      <inertia ixx="0.154692" ixy="-0.0" ixz="0.0" iyy="0.23723" iyz="-0.0" izz="0.154692"/>
-    </inertial>
-    <visual>
-      <origin rpy="0 0 0" xyz="-0.7524 0.281125 0.244"/>
-      <geometry>
-        <mesh filename="package://robot_description/meshes/wheel_3.stl" scale="0.001 0.001 0.001"/>
-      </geometry>
-      <material name="silver"/>
-    </visual>
-    <collision>
-      <origin rpy="0 0 0" xyz="-0.7524 0.281125 0.244"/>
-      <geometry>
-        <mesh filename="package://robot_description/meshes/wheel_3.stl" scale="0.001 0.001 0.001"/>
-      </geometry>
-    </collision>
-  </link>
-  <link name="wheel_2">
-    <inertial>
-      <origin rpy="0 0 0" xyz="-1.609823385706477e-15 -0.05499999999999988 1.3877787807814457e-16"/>
-      <mass value="35.77866096632706"/>
-      <inertia ixx="0.154692" ixy="0.0" ixz="0.0" iyy="0.23723" iyz="-0.0" izz="0.154692"/>
-    </inertial>
-    <visual>
-      <origin rpy="0 0 0" xyz="-0.3624 0.281125 0.244"/>
-      <geometry>
-        <mesh filename="package://robot_description/meshes/wheel_2.stl" scale="0.001 0.001 0.001"/>
-      </geometry>
-      <material name="silver"/>
-    </visual>
-    <collision>
-      <origin rpy="0 0 0" xyz="-0.3624 0.281125 0.244"/>
-      <geometry>
-        <mesh filename="package://robot_description/meshes/wheel_2.stl" scale="0.001 0.001 0.001"/>
-      </geometry>
-    </collision>
-  </link>
-  <link name="wheel_1">
-    <inertial>
-      <origin rpy="0 0 0" xyz="-1.7208456881689926e-15 -0.05499999999999988 1.1102230246251565e-16"/>
-      <mass value="35.77866096632706"/>
-      <inertia ixx="0.154692" ixy="-0.0" ixz="0.0" iyy="0.23723" iyz="-0.0" izz="0.154692"/>
-    </inertial>
-    <visual>
-      <origin rpy="0 0 0" xyz="0.1376 0.281125 0.244"/>
-      <geometry>
-        <mesh filename="package://robot_description/meshes/wheel_1.stl" scale="0.001 0.001 0.001"/>
-      </geometry>
-      <material name="silver"/>
-    </visual>
-    <collision>
-      <origin rpy="0 0 0" xyz="0.1376 0.281125 0.244"/>
-      <geometry>
-        <mesh filename="package://robot_description/meshes/wheel_1.stl" scale="0.001 0.001 0.001"/>
-      </geometry>
-    </collision>
-  </link>
-  <link name="wheel_r_1">
-    <inertial>
-      <origin rpy="0 0 0" xyz="-1.7208456881689926e-15 0.05499999999999988 1.942890293094024e-16"/>
+      <origin rpy="0 0 0" xyz="-1.4432899320127035e-15 0.05499999999999988 4.440892098500626e-16"/>
       <mass value="35.77866096632706"/>
       <inertia ixx="0.154692" ixy="0.0" ixz="0.0" iyy="0.23723" iyz="0.0" izz="0.154692"/>
     </inertial>
     <visual>
-      <origin rpy="0 0 0" xyz="0.1376 -0.281125 0.244"/>
-      <geometry>
-        <mesh filename="package://robot_description/meshes/wheel_r_1.stl" scale="0.001 0.001 0.001"/>
-      </geometry>
-      <material name="silver"/>
-    </visual>
-    <collision>
-      <origin rpy="0 0 0" xyz="0.1376 -0.281125 0.244"/>
-      <geometry>
-        <mesh filename="package://robot_description/meshes/wheel_r_1.stl" scale="0.001 0.001 0.001"/>
-      </geometry>
-    </collision>
-  </link>
-  <link name="wheel_r_2">
-    <inertial>
-      <origin rpy="0 0 0" xyz="-1.609823385706477e-15 0.05499999999999988 2.220446049250313e-16"/>
-      <mass value="35.77866096632706"/>
-      <inertia ixx="0.154692" ixy="-0.0" ixz="0.0" iyy="0.23723" iyz="0.0" izz="0.154692"/>
-    </inertial>
-    <visual>
-      <origin rpy="0 0 0" xyz="-0.3624 -0.281125 0.244"/>
-      <geometry>
-        <mesh filename="package://robot_description/meshes/wheel_r_2.stl" scale="0.001 0.001 0.001"/>
-      </geometry>
-      <material name="silver"/>
-    </visual>
-    <collision>
-      <origin rpy="0 0 0" xyz="-0.3624 -0.281125 0.244"/>
-      <geometry>
-        <mesh filename="package://robot_description/meshes/wheel_r_2.stl" scale="0.001 0.001 0.001"/>
-      </geometry>
-    </collision>
-  </link>
-  <link name="wheel_r_3">
-    <inertial>
-      <origin rpy="0 0 0" xyz="-1.4432899320127035e-15 0.05499999999999988 4.440892098500626e-16"/>
-      <mass value="35.77866096632706"/>
-      <inertia ixx="0.154692" ixy="0.0" ixz="0.0" iyy="0.23723" iyz="0.0" izz="0.154692"/>
-    </inertial>
-    <visual>
       <origin rpy="0 0 0" xyz="-0.7524 -0.281125 0.244"/>
       <geometry>
@@ -234,28 +235,58 @@
   </link>
   <joint name="Revolute 1" type="fixed">
-    <origin rpy="0 0 0" xyz="0.3024 -0.243025 0.0"/>
+    <origin rpy="0 0 0" xyz="-0.06 -0.243025 0.244"/>
+    <parent link="base_link"/>
+    <child link="suspension_1_right_1"/>
+    <axis xyz="0.0 1.0 0.0"/>
+  </joint>
+  <joint name="Revolute 2" type="fixed">
+    <origin rpy="0 0 0" xyz="-0.06 0.243025 0.244"/>
     <parent link="base_link"/>
     <child link="suspension_1_left_1"/>
     <axis xyz="0.0 1.0 0.0"/>
   </joint>
-  <joint name="Revolute 2" type="fixed">
-    <origin rpy="0 0 0" xyz="0.3024 0.243025 0.0"/>
-    <parent link="base_link"/>
-    <child link="suspension_1_right_1"/>
-    <axis xyz="0.0 1.0 0.0"/>
-  </joint>
   <joint name="Revolute 3" type="fixed">
     <origin rpy="0 0 0" xyz="0.3 -0.0381 -0.122"/>
+    <parent link="suspension_1_right_1"/>
+    <child link="suspension_2_right_1"/>
+    <axis xyz="0.0 1.0 0.0"/>
+  </joint>
+  <joint name="Revolute 4" type="fixed">
+    <origin rpy="0 0 0" xyz="0.3 0.0381 -0.122"/>
     <parent link="suspension_1_left_1"/>
     <child link="suspension_2_left_1"/>
-    <axis xyz="0.0 1.0 0.0"/>
-  </joint>
-  <joint name="Revolute 4" type="fixed">
-    <origin rpy="0 0 0" xyz="0.3 0.0381 -0.122"/>
+    <axis xyz="0.0 -1.0 0.0"/>
+  </joint>
+  <joint name="joint_wheel_r1" type="continuous">
+    <origin rpy="0 0 0" xyz="0.15 0.0 -0.122"/>
+    <parent link="suspension_2_right_1"/>
+    <child link="wheel_r_3"/>
+    <axis xyz="0.0 1.0 0.0"/>
+  </joint>
+  <joint name="joint_wheel_r2" type="continuous">
+    <origin rpy="0 0 0" xyz="-0.24 0.0 -0.122"/>
+    <parent link="suspension_2_right_1"/>
+    <child link="wheel_r_2"/>
+    <axis xyz="0.0 1.0 0.0"/>
+  </joint>
+  <joint name="joint_wheel_r3" type="continuous">
+    <origin rpy="0 0 0" xyz="-0.44 -0.0381 -0.244"/>
     <parent link="suspension_1_right_1"/>
-    <child link="suspension_2_right_1"/>
-    <axis xyz="0.0 -1.0 0.0"/>
-  </joint>
-  <joint name="joint_wheel_r1" type="continuous">
+    <child link="wheel_r_1"/>
+    <axis xyz="0.0 1.0 0.0"/>
+  </joint>
+  <joint name="joint_wheel_l1" type="continuous">
+    <origin rpy="0 0 0" xyz="-0.44 0.0381 -0.244"/>
+    <parent link="suspension_1_left_1"/>
+    <child link="wheel_1"/>
+    <axis xyz="0.0 1.0 0.0"/>
+  </joint>
+  <joint name="joint_wheel_l2" type="continuous">
+    <origin rpy="0 0 0" xyz="-0.24 0.0 -0.122"/>
+    <parent link="suspension_2_left_1"/>
+    <child link="wheel_2"/>
+    <axis xyz="0.0 1.0 0.0"/>
+  </joint>
+  <joint name="joint_wheel_l3" type="continuous">
     <origin rpy="0 0 0" xyz="0.15 0.0 -0.122"/>
     <parent link="suspension_2_left_1"/>
@@ -263,33 +294,3 @@
     <axis xyz="0.0 1.0 0.0"/>
   </joint>
-  <joint name="joint_wheel_r2" type="continuous">
-    <origin rpy="0 0 0" xyz="-0.24 0.0 -0.122"/>
-    <parent link="suspension_2_left_1"/>
-    <child link="wheel_2"/>
-    <axis xyz="0.0 1.0 0.0"/>
-  </joint>
-  <joint name="joint_wheel_r3" type="continuous">
-    <origin rpy="0 0 0" xyz="-0.44 -0.0381 -0.244"/>
-    <parent link="suspension_1_left_1"/>
-    <child link="wheel_1"/>
-    <axis xyz="0.0 1.0 0.0"/>
-  </joint>
-  <joint name="joint_wheel_l1" type="continuous">
-    <origin rpy="0 0 0" xyz="-0.44 0.0381 -0.244"/>
-    <parent link="suspension_1_right_1"/>
-    <child link="wheel_r_1"/>
-    <axis xyz="0.0 1.0 0.0"/>
-  </joint>
-  <joint name="joint_wheel_l2" type="continuous">
-    <origin rpy="0 0 0" xyz="-0.24 0.0 -0.122"/>
-    <parent link="suspension_2_right_1"/>
-    <child link="wheel_r_2"/>
-    <axis xyz="0.0 1.0 0.0"/>
-  </joint>
-  <joint name="joint_wheel_l3" type="continuous">
-    <origin rpy="0 0 0" xyz="0.15 0.0 -0.122"/>
-    <parent link="suspension_2_right_1"/>
-    <child link="wheel_r_3"/>
-    <axis xyz="0.0 1.0 0.0"/>
-  </joint>
 </robot>

File: ros2_ws/src/robot_description/urdf/robot_gz.urdf.xacro (robot description, xacro)
@@ -8,8 +8,11 @@
         <xacro:white/>
     </gazebo>
+    <gazebo reference="suspension_1_right_1">
+        <xacro:dark_grey/>
+    </gazebo>
     <gazebo reference="suspension_1_left_1">
         <xacro:dark_grey/>
     </gazebo>
-    <gazebo reference="suspension_1_right_1">
+    <gazebo reference="suspension_2_right_1">
         <xacro:dark_grey/>
     </gazebo>
@@ -17,8 +20,14 @@
         <xacro:dark_grey/>
     </gazebo>
-    <gazebo reference="suspension_2_right_1">
-        <xacro:dark_grey/>
+    <gazebo reference="wheel_r_3">
+        <xacro:black/>
     </gazebo>
-    <gazebo reference="wheel_3">
+    <gazebo reference="wheel_r_2">
+        <xacro:black/>
+    </gazebo>
+    <gazebo reference="wheel_r_1">
+        <xacro:black/>
+    </gazebo>
+    <gazebo reference="wheel_1">
         <xacro:black/>
     </gazebo>
@@ -26,14 +35,5 @@
         <xacro:black/>
     </gazebo>
-    <gazebo reference="wheel_1">
-        <xacro:black/>
-    </gazebo>
-    <gazebo reference="wheel_r_1">
-        <xacro:black/>
-    </gazebo>
-    <gazebo reference="wheel_r_2">
-        <xacro:black/>
-    </gazebo>
-    <gazebo reference="wheel_r_3">
+    <gazebo reference="wheel_3">
         <xacro:black/>
     </gazebo>
@@ -48,11 +48,17 @@
             <wheel_separation>.67</wheel_separation>
             <wheel_radius>.22</wheel_radius>
-            <max_wheel_torque>200</max_wheel_torque>
-            <max_wheel_acceleration>10.0</max_wheel_acceleration>
-            <odometry_frame>odom</odometry_frame>
-            <robot_base_frame>base_link</robot_base_frame>
-            <publish_odom>true</publish_odom>
-            <publish_odom_tf>true</publish_odom_tf>
-            <publish_wheel_tf>true</publish_wheel_tf>
+            <odom_publish_frequency>50</odom_publish_frequency>
+            <frame_id>odom</frame_id>
+            <child_frame_id>base_footprint</child_frame_id>
+        </plugin>
+    </gazebo>
+    <gazebo>
+        <plugin name="ignition::gazebo::systems::JointStatePublisher" filename="libignition-gazebo-joint-state-publisher-system.so">
+            <joint_name>joint_wheel_r1</joint_name>
+            <joint_name>joint_wheel_r2</joint_name>
+            <joint_name>joint_wheel_r3</joint_name>
+            <joint_name>joint_wheel_l1</joint_name>
+            <joint_name>joint_wheel_l2</joint_name>
+            <joint_name>joint_wheel_l3</joint_name>
         </plugin>
     </gazebo>
