Commit message: feat(B-002): change depth cam to rgb depth cam in gz sim, now working

File: ros2_ws/src/robot_description/urdf/macros.xacro (robot description, xacro)
@@ -37,8 +37,11 @@
         </visual>
     </xacro:macro>
-    <xacro:property name="zed_width" value="640" />
-    <xacro:property name="zed_height" value="480" />
-    <xacro:property name="zed_horizontal_fov" value="1.089" />
-    <xacro:property name="zed_fx" value="${zed_width / (2 * (sin(zed_horizontal_fov / 2) / cos(zed_horizontal_fov / 2)))}" />
+    <xacro:property name="zed_width" value="1280" />
+    <xacro:property name="zed_height" value="720" />
+    <xacro:property name="zed_horizontal_fov_deg" value="120" />
+    <xacro:property name="zed_horizontal_fov" value="${zed_horizontal_fov_deg * pi / 180.0}" />
+    <xacro:property name="zed_fx" value="${zed_width / (2 * tan(zed_horizontal_fov / 2))}" />
     <xacro:property name="zed_fy" value="${zed_fx}" />
+    <xacro:property name="zed_cx" value="${zed_width / 2.0}" />
+    <xacro:property name="zed_cy" value="${zed_height / 2.0}" />
 </robot>

File: ros2_ws/src/robot_description/urdf/robot_gz.urdf.xacro (robot description, xacro)
@@ -39,27 +39,52 @@
     </gazebo>
     <gazebo reference="camera_link">
-        <xacro:orange/>
-        <sensor name="camera" type="depth_camera">
-            <pose> 0 0 0 0 0 0</pose>
-            <always_on>1</always_on>
-            <visualize>1</visualize>
-            <update_rate>10</update_rate>
-            <topic>/depth_cam</topic>
-            <gz_frame_id>camera_link_optical</gz_frame_id>
-            <camera>
-                <camera_info_topic>/depth_cam/camera_info</camera_info_topic>
-                <horizontal_fov>${zed_horizontal_fov}</horizontal_fov>
-                <image>
-                    <format>R8G8B8</format>
-                    <width>${zed_width}</width>
-                    <height>${zed_height}</height>
-                </image>
-                <clip>
-                    <near>0.01</near>
-                    <far>100.0</far>
-                </clip>
-            </camera>
-        </sensor>
-    </gazebo>
+  <sensor name="zed2i" type="rgbd_camera">
+    <ignition_frame_id>camera_link</ignition_frame_id>
+    <camera name="zed2i">
+      <horizontal_fov>${zed_horizontal_fov}</horizontal_fov>
+      <lens>
+        <intrinsics>
+          <fx>${zed_fx}</fx>
+          <fy>${zed_fy}</fy>
+          <cx>${zed_cx}</cx>
+          <cy>${zed_cy}</cy>
+          <s>0</s>
+        </intrinsics>
+      </lens>
+      <distortion>
+        <k1>0.104207</k1>
+        <k2>-0.255558</k2>
+        <k3>0.128694</k3>
+        <p1>0.000512</p1>
+        <p2>0.000319</p2>
+        <center>0.5 0.5</center>
+      </distortion>
+      <image>
+        <width>${zed_width}</width>
+        <height>${zed_height}</height>
+        <format>L8</format>
+      </image>
+      <clip>
+        <near>0.01</near>
+        <far>300</far>
+      </clip>
+      <depth_camera>
+        <clip>
+          <near>0.1</near>
+          <far>10</far>
+        </clip>
+      </depth_camera>
+      <noise>
+        <type>gaussian</type>
+        <mean>0</mean>
+        <stddev>0.003</stddev>
+      </noise>
+    </camera>
+    <always_on>1</always_on>
+    <update_rate>10</update_rate>
+    <visualize>0</visualize>
+    <topic>/depth_cam</topic>
+  </sensor>
+</gazebo>
     <gazebo>
         <!-- Render and publish camera / GPU sensor data for this spawned model. -->
