Commit message: add depth cam work so far

File: ros2_ws/src/robot_description/urdf/camera.urdf.xacro (robot description, xacro)
@@ -4,5 +4,5 @@
             <parent link="base_link"/>
             <child link="camera_link"/>
-            <origin xyz="0.3624 0.0 0.1" rpy="0.0 0.0 0.0"/>
+            <origin xyz="0.3624 0.0 0.3524" rpy="0.0 0.0 0.0"/>
         </joint>
         <joint name="camera_optical_joint" type="fixed">
@@ -14,5 +14,5 @@
             <visual>
                     <geometry>
-                        <box size=".010 .03 0.03"/>
+                        <box size=".0303 .1753 0.0431"/>
                     </geometry>
                     <material name="silver">

File: ros2_ws/src/robot_description/urdf/macros.xacro (robot description, xacro)
@@ -37,3 +37,8 @@
         </visual>
     </xacro:macro>
+    <xacro:property name="zed_width" value="640" />
+    <xacro:property name="zed_height" value="480" />
+    <xacro:property name="zed_horizontal_fov" value="1.089" />
+    <xacro:property name="zed_fx" value="${zed_width / (2 * (sin(zed_horizontal_fov / 2) / cos(zed_horizontal_fov / 2)))}" />
+    <xacro:property name="zed_fy" value="${zed_fx}" />
 </robot>

File: ros2_ws/src/robot_description/urdf/robot_gz.urdf.xacro (robot description, xacro)
@@ -40,25 +40,22 @@
     <gazebo reference="camera_link">
         <xacro:orange/>
-        <sensor name="camera" type="camera">
+        <sensor name="camera" type="depth_camera">
             <pose> 0 0 0 0 0 0</pose>
-            <always_on>true</always_on>
-            <visualize>true</visualize>
+            <always_on>1</always_on>
+            <visualize>1</visualize>
             <update_rate>10</update_rate>
-            <topic>/camera/image_raw</topic>
-            <!-- Match image headers to the URDF frame published by
-                 robot_state_publisher; avoids a Gazebo-specific static TF. -->
+            <topic>/depth_cam</topic>
             <gz_frame_id>camera_link_optical</gz_frame_id>
             <camera>
-                <camera_info_topic>/camera/camera_info</camera_info_topic>
-                <optical_frame_id>camera_link_optical</optical_frame_id>
-                <horizontal_fov>1.089</horizontal_fov>
+                <camera_info_topic>/depth_cam/camera_info</camera_info_topic>
+                <horizontal_fov>${zed_horizontal_fov}</horizontal_fov>
                 <image>
                     <format>R8G8B8</format>
-                    <width>640</width>
-                    <height>480</height>
+                    <width>${zed_width}</width>
+                    <height>${zed_height}</height>
                 </image>
                 <clip>
-                    <near>0.05</near>
-                    <far>8.0</far>
+                    <near>0.01</near>
+                    <far>100.0</far>
                 </clip>
             </camera>

Commit message: feat(B-002): add zed2i cam

File: ros2_ws/src/robot_description/urdf/camera.urdf.xacro (robot description, xacro)
@@ -4,5 +4,5 @@
             <parent link="base_link"/>
             <child link="camera_link"/>
-            <origin xyz="0.3624 0.0 0.3524" rpy="0.0 0.0 0.0"/>
+            <origin xyz="0.3624 0.0 0.3424" rpy="0.0 0.0 0.0"/>
         </joint>
         <joint name="camera_optical_joint" type="fixed">
@@ -13,6 +13,8 @@
         <link name="camera_link">
             <visual>
+                    <origin xyz="0.0 0.0 0.0" rpy="0 0 ${pi/2}"/>
                     <geometry>
-                        <box size=".0303 .1753 0.0431"/>
+                        <mesh filename="package://robot_description/meshes/zed2i.stl" scale="1.0 1.0 1.0"/>
+                        <!--box size=".0303 .1753 0.0431"/!-->
                     </geometry>
                     <material name="silver">

File: ros2_ws/src/robot_description/urdf/robot_gz.urdf.xacro (robot description, xacro)
@@ -39,52 +39,53 @@
     </gazebo>
     <gazebo reference="camera_link">
-  <sensor name="zed2i" type="rgbd_camera">
-    <ignition_frame_id>camera_link</ignition_frame_id>
-    <camera name="zed2i">
-      <horizontal_fov>${zed_horizontal_fov}</horizontal_fov>
-      <lens>
-        <intrinsics>
-          <fx>${zed_fx}</fx>
-          <fy>${zed_fy}</fy>
-          <cx>${zed_cx}</cx>
-          <cy>${zed_cy}</cy>
-          <s>0</s>
-        </intrinsics>
-      </lens>
-      <distortion>
-        <k1>0.104207</k1>
-        <k2>-0.255558</k2>
-        <k3>0.128694</k3>
-        <p1>0.000512</p1>
-        <p2>0.000319</p2>
-        <center>0.5 0.5</center>
-      </distortion>
-      <image>
-        <width>${zed_width}</width>
-        <height>${zed_height}</height>
-        <format>L8</format>
-      </image>
-      <clip>
-        <near>0.01</near>
-        <far>300</far>
-      </clip>
-      <depth_camera>
-        <clip>
-          <near>0.1</near>
-          <far>10</far>
-        </clip>
-      </depth_camera>
-      <noise>
-        <type>gaussian</type>
-        <mean>0</mean>
-        <stddev>0.003</stddev>
-      </noise>
-    </camera>
-    <always_on>1</always_on>
-    <update_rate>10</update_rate>
-    <visualize>0</visualize>
-    <topic>/depth_cam</topic>
-  </sensor>
-</gazebo>
+        <xacro:black/>
+        <sensor name="zed2i" type="rgbd_camera">
+            <ignition_frame_id>camera_link</ignition_frame_id>
+            <camera name="zed2i">
+            <horizontal_fov>${zed_horizontal_fov}</horizontal_fov>
+            <lens>
+                <intrinsics>
+                <fx>${zed_fx}</fx>
+                <fy>${zed_fy}</fy>
+                <cx>${zed_cx}</cx>
+                <cy>${zed_cy}</cy>
+                <s>0</s>
+                </intrinsics>
+            </lens>
+            <distortion>
+                <k1>0.104207</k1>
+                <k2>-0.255558</k2>
+                <k3>0.128694</k3>
+                <p1>0.000512</p1>
+                <p2>0.000319</p2>
+                <center>0.5 0.5</center>
+            </distortion>
+            <image>
+                <width>${zed_width}</width>
+                <height>${zed_height}</height>
+                <format>L8</format>
+            </image>
+            <clip>
+                <near>0.01</near>
+                <far>300</far>
+            </clip>
+            <depth_camera>
+                <clip>
+                <near>0.1</near>
+                <far>10</far>
+                </clip>
+            </depth_camera>
+            <noise>
+                <type>gaussian</type>
+                <mean>0</mean>
+                <stddev>0.003</stddev>
+            </noise>
+            </camera>
+            <always_on>1</always_on>
+            <update_rate>10</update_rate>
+            <visualize>0</visualize>
+            <topic>/depth_cam</topic>
+        </sensor>
+    </gazebo>
     <gazebo>
         <!-- Render and publish camera / GPU sensor data for this spawned model. -->
