Commit message: robot_description: make use_sim a settable xacro:arg
Replaces the hardcoded <xacro:property name="use_sim" value="true"/> with a
<xacro:arg name="use_sim" default="true"/> plus a property mirror, so the
ros2_control backend is selectable from a launch file (xacro ... use_sim:=false)
while every downstream ${use_sim} reference keeps working. Default stays true,
so sim_gz.launch.py (which passes no arg) is byte-for-byte unchanged.

robot_gz.urdf.xacro is left included unconditionally on purpose - its <gazebo>
blocks are inert outside Gazebo, so gating it only risks the working sim.

Co-Authored-By: Claude Sonnet 5 <noreply@anthropic.com>

File: ros2_ws/src/robot_description/urdf/robot.urdf.xacro (robot description, xacro)
@@ -1,6 +1,16 @@
 <?xml version="1.0" ?>
 <robot name="robot" xmlns:xacro="http://www.ros.org/wiki/xacro" >
-    <xacro:property name="use_sim" value="true"/>
+    <!-- use_sim selects the ros2_control backend (Gazebo ign_ros2_control vs the
+         real OdescSystemHardware CAN driver). Settable from a launch file:
+             xacro robot.urdf.xacro use_sim:=false
+         Default is true, so sim_gz.launch.py (which passes no arg) is unchanged.
+         The property mirror keeps every downstream ${use_sim} reference working. -->
+    <xacro:arg name="use_sim" default="true"/>
+    <xacro:property name="use_sim" value="$(arg use_sim)"/>
     <xacro:include filename="robot_core.urdf.xacro"/>
+    <!-- robot_gz.urdf.xacro is left included unconditionally: its <gazebo> blocks
+         are inert outside Gazebo (robot_state_publisher and a standalone
+         controller_manager both ignore them), so gating it buys nothing and only
+         risks the confirmed-working sim expansion. -->
     <xacro:include filename="robot_gz.urdf.xacro"/>
     <xacro:include filename="camera.urdf.xacro"/>
